File: RP2350-Micro-Devboard.kicad_pcb (KiCad board)
At the start: 2 copper layers, 18.5 x 25.8 mm, 31 parts, among them J1 USB_C_Receptacle_USB2.0_14P, J2 Conn_01x07, J3 Conn_01x07, SW2 SW_Push, U1 MCP1700x-330xxTT, U2 RP2350_60QFN, Y1 12MHz

Commit message: first completion of shitty routing
Parts:
- removed J1: USB_C_Receptacle_USB2.0_14P, Connector_USB:USB_C_Receptacle_HRO_TYPE-C-31-M-12
- removed R1, R2: 5.1k, Resistor_SMD:R_0402_1005Metric
- added J4: USB_B_Micro, RP2350_60QFN_minimal:USB_Micro-B_Amphenol_10103594-0001LF_Horizontal_modified, F.Cu at (153.3, 56.9)
- C1, C10: moved to F.Cu
- C17, SW2: moved to B.Cu
- moved J3 49.6 mm to (161.1, 74.7), turned to 180 degrees
- moved C3 49.3 mm to (158.2, 64.9), turned to 45 degrees
- moved C4 49.2 mm to (156.2, 62.6), turned to 90 degrees
- moved C2 49.0 mm to (155.9, 73.2), turned to 180 degrees
- moved SW2 48.8 mm to (156.0, 74.4), turned to 90 degrees
- moved C7 48.2 mm to (157.8, 70.4), turned to -90 degrees
- moved C11 47.2 mm to (152.1, 62.9), turned to -90 degrees
- moved C10 45.4 mm to (158.7, 70.4), turned to -90 degrees
- moved C13 44.0 mm to (148.6, 76.2)
- moved U1 44.0 mm to (149.4, 62.7), turned to 0 degrees
- moved R8 43.9 mm to (158.8, 61.1), turned to 90 degrees
- moved C15 43.9 mm to (158.8, 63.0)
- moved C6 43.8 mm to (148.0, 71.0), turned to -135 degrees
- moved Y1 43.5 mm to (151.2, 75.4)
- moved R5 43.4 mm to (153.8, 74.6)
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Connections:
- J2 pad 1: /GPIO26 -> /GPIO0
- J2 pad 2: /GPIO27 -> /GPIO1
- J2 pad 3: /GPIO28 -> /GPIO2
- J2 pad 4: /GPIO5 -> /GPIO3
- J2 pad 5: /GPIO6 -> /GPIO4
- J2 pad 6: /GPIO7 -> /GPIO5
- J2 pad 7: /GPIO0 -> /GPIO6
- J3 pad 1: /GPIO1 -> /GPIO7
- J3 pad 2: /GPIO2 -> /GPIO26
- J3 pad 3: /GPIO4 -> /GPIO27
- J3 pad 4: /GPIO3 -> /GPIO28
Routing:
- net /GPIO26: track 49.5 -> 6.84 mm, vias 2 -> 0
- net GND: track 45.4 -> 75.9 mm, vias 0 -> 7
- net /GPIO28: track 34.0 -> 4.55 mm, vias 1 -> 0
- net /GPIO27: track 33.8 -> 5.43 mm, vias 3 -> 0
- net /VBUS: track 44.4 -> 16.1 mm, vias 3 -> 2
- net /GPIO2: track 33.3 -> 5.71 mm, vias 1 -> 0
- net +3V3: track 46.5 -> 71.7 mm, vias 1 -> 6
- net Net-(U2-RUN): track 21.3 -> 3.30 mm, vias 2 -> 1
- net /GPIO3: track 22.8 -> 4.84 mm, vias 1 -> 0
- net /GPIO4: track 22.8 -> 5.15 mm, vias 2 -> 0
- net +1V1: track 39.9 -> 29.7 mm, vias 5 -> 2
- net Net-(J1-CC1): track 9.55 -> 0.00 mm
- net /GPIO7: track 7.41 -> 16.1 mm, vias 0 -> 1
- net Net-(J1-CC2): track 7.72 -> 0.00 mm
- net /USB_D-: track 11.1 -> 3.35 mm
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- added copper zone on B.Cu, net GND
- added copper zone on F.Cu, net GND
- removed copper zone on B.Cu, net (none)
- removed copper zone on F.Cu, net (none)
Other:
- board size 18.5 x 25.8 mm -> 19.5 x 22.2 mm

Commit message: fix the drc
Parts:
- moved C3 0.06 mm to (158.3, 64.9)
Routing:
- net GND: track 75.9 -> 86.1 mm, vias 7 -> 9
Other:
- board size 19.5 x 22.2 mm -> 19.5 x 22.6 mm
